File: ergogen/output/pcbs/main/dofeKeyboard_main.kicad_pcb (KiCad board)
At the start: 2 copper layers, 119.2 x 87.6 mm, 40 parts

Commit message: updated pcb + another image
Routing:
- net R3: track 69.7 -> 71.4 mm
- net C1: track 217.2 -> 218.4 mm
- net C0: track 236.7 -> 237.9 mm
- net C2: track 204.0 -> 202.9 mm
- net C3: track 184.1 -> 184.7 mm
